Commit message: allow lidar to be rotated since in my build I prefer the motor of the lidar to be on the back

File: description/turbopi.urdf.xacro (robot description, xacro)
@@ -5,4 +5,5 @@
 	<xacro:arg name="use_camera" default="default" />
 	<xacro:arg name="use_lidar" default="default" />
+	<xacro:arg name="lidar_yaw" default="${pi}" />
 	<xacro:arg name="use_version" default="8" />
 	<xacro:include filename="colors.xacro" />
@@ -13,5 +14,5 @@
                         use_camera="$(arg use_camera)" />
 	<xacro:camera use_camera="$(arg use_camera)" />
-	<xacro:lidar use_lidar="$(arg use_lidar)" />
+	<xacro:lidar use_lidar="$(arg use_lidar)" lidar_yaw="$(arg lidar_yaw)" />
     <xacro:macro name="gazebo" params="use_hardware">
       <xacro:if value="${use_hardware == 'ign_gazebo'}">

File: description/turbopi_core.xacro (robot description, xacro)
@@ -312,5 +312,8 @@
     </link>
     <!-- 360 Lidar -->
-    <xacro:macro name="lidar" params="use_lidar">
+    <!-- lidar_yaw: rotation around Z axis for the lidar mount.
+         Default is pi (180°) because the RPLidar A1 is mounted facing backward
+         on the TurboPi. Set lidar_yaw:=0 if your mount faces forward. -->
+    <xacro:macro name="lidar" params="use_lidar lidar_yaw:=${pi}">
         <xacro:if value="${use_lidar == 'lidar'}">
             <joint name="lidar_joint" type="fixed">
@@ -318,5 +321,5 @@
                 <child link="lidar"/>
                 <axis xyz="0 0 1"/>
-                <origin xyz="${-lidar_length/2 + 0.01} 0 0.0725" rpy="0 0 0"/>
+                <origin xyz="${-lidar_length/2 + 0.01} 0 0.0725" rpy="0 0 ${lidar_yaw}"/>
             </joint>
             <link name="lidar">
